File: 4MD/4MD.sch (KiCad schematic (older format))
At the start: 10 parts, among them J1 Signal_In, J2 Signal_Out, Q1 2N2219

Commit message: Izlabots 4MD
Changed lines of the file:
@@
 	1    0    0    -1
 $EndComp
+$Comp
+L power:PWR_FLAG #FLG0101
+U 1 1 5CEF7BE2
+P 4850 1850
+F 0 "#FLG0101" H 4850 1925 50  0001 C CNN
+F 1 "PWR_FLAG" H 4850 2024 50  0000 C CNN
+F 2 "" H 4850 1850 50  0001 C CNN
+F 3 "~" H 4850 1850 50  0001 C CNN
+	1    4850 1850
+	1    0    0    -1
+$EndComp
+Connection ~ 4850 1850
+$Comp
+L power:PWR_FLAG #FLG0102
+U 1 1 5CEF7C18
+P 4850 3700
+F 0 "#FLG0102" H 4850 3775 50  0001 C CNN
+F 1 "PWR_FLAG" H 4850 3873 50  0000 C CNN
+F 2 "" H 4850 3700 50  0001 C CNN
+F 3 "~" H 4850 3700 50  0001 C CNN
+	1    4850 3700
+	-1   0    0    1
+$EndComp
+Connection ~ 4850 3700
 $EndSCHEMATC
